File: EagleCAD/ReflowMaster.sch (EAGLE design)
At the start: 42 parts, among them Q1 600mA/40V, SW1 SPST_TACT-KMR2, X2 32.768

Commit message: added a programming header + PCB tweaks
Parts:
- removed R1: 100k, microbuilder:RESISTOR0805_NOOUTLINE
- added J3: (no value), SparkFun-Connectors:CONN_05NO_SILK
Connections:
- removed net EN: LDO.EN, R1.2
- new net VBUS_SW: C6.1, D1.C, FAN.1, LDO.EN, LDO.IN, R2.1, R3.1, SWITCH.2, TFT.1
- net !RESET: now also J3.5
- net +3V3: now also J3.2
- net GND: now also J3.1
- net SWCLK: now also J3.4
- net SWDIO: now also J3.3
- net VBUS: no longer C6.1, D1.C, FAN.1, LDO.IN, R1.1, R2.1, R3.1, SWITCH.2, TFT.1
Other:
- note added: "PROGAMMING"
- moved on the sheet: C14
